Commit message: simulator error fixed

File: keti_sdk_simulator/keti_robot_moveit_config/config/gazebo_keti_robot_description.urdf (robot description, URDF)
Before this commit: robot keti_robot_description, 22 links, 21 joints
Joints:
- joint world_base: origin xyz=0 0 0 rpy=0 0 0 -> xyz=0 0 0.803 rpy=0 0 0
