Commit message: simulator orientation 수정

File: keti_sdk_simulator/keti_robot_description/urdf/keti_robot_description.urdf (robot description, URDF)
Before this commit: robot keti_robot_description, 16 links, 15 joints
Joints:
- joint link6_gripper_fixed: limit lower=-3.15 upper=3.15 effort=10 velocity=100 -> lower=-6.15 upper=6.15 effort=10 velocity=100
- joint q1: limit lower=-3.15 upper=3.15 effort=10 velocity=100 -> lower=-6.15 upper=6.15 effort=10 velocity=100
- joint q2: limit lower=-3.15 upper=3.15 effort=10 velocity=100 -> lower=-6.15 upper=6.15 effort=10 velocity=100
- joint q3: limit lower=-3.15 upper=3.15 effort=10 velocity=100 -> lower=-6.15 upper=6.15 effort=10 velocity=100
- joint q4: limit lower=-3.15 upper=3.15 effort=10 velocity=100 -> lower=-6.15 upper=6.15 effort=10 velocity=100
- joint q5: limit lower=-3.15 upper=3.15 effort=10 velocity=100 -> lower=-6.15 upper=6.15 effort=10 velocity=100
- joint q6: limit lower=-3.15 upper=3.15 effort=10 velocity=100 -> lower=-6.15 upper=6.15 effort=10 velocity=100

Commit message: simulator camera view 및 ui 추가

File: keti_sdk_simulator/keti_robot_description/urdf/keti_robot_description.urdf (robot description, URDF)
Before this commit: robot keti_robot_description, 16 links, 15 joints
Links:
- removed link obstacle
- removed link plate_pick
- removed link plate_place
- added link cam, mass 0.0224324424296924; collision mesh filename=package://keti_robot_description/meshes/cam.STL; visual mesh filename=package://keti_robot_description/meshes/cam.STL
- added link pick, mass 4.07592; collision mesh filename=package://keti_robot_description/meshes/pick.STL; visual mesh filename=package://keti_robot_description/meshes/pick.STL
- added link pick_circle, mass 0.0441236688196687; collision mesh filename=package://keti_robot_description/meshes/pick_circle.STL; visual mesh filename=package://keti_robot_description/meshes/pick_circle.STL
- added link pick_cross, mass 0.0400000000000002; collision mesh filename=package://keti_robot_description/meshes/pick_cross.STL; visual mesh filename=package://keti_robot_description/meshes/pick_cross.STL
- added link pick_rectangle, mass 0.0442885009851994; collision mesh filename=package://keti_robot_description/meshes/pick_rectangle.STL; visual mesh filename=package://keti_robot_description/meshes/pick_rectangle.STL
- added link place, mass 0.785447283360145; collision mesh filename=package://keti_robot_description/meshes/place.STL; visual mesh filename=package://keti_robot_description/meshes/place.STL
- added link place_circle, mass 0.0577456825709279; collision mesh filename=package://keti_robot_description/meshes/place_circle.STL; visual mesh filename=package://keti_robot_description/meshes/place_circle.STL
- added link place_cross, mass 0.0578280000000003; collision mesh filename=package://keti_robot_description/meshes/place_cross.STL; visual mesh filename=package://keti_robot_description/meshes/place_cross.STL
- added link place_rectangle, mass 0.0418280000000002; collision mesh filename=package://keti_robot_description/meshes/place_rectangle.STL; visual mesh filename=package://keti_robot_description/meshes/place_rectangle.STL
- added link table, mass 361.6; collision mesh filename=package://keti_robot_description/meshes/table.STL; visual mesh filename=package://keti_robot_description/meshes/table.STL
- link base: mass 1166.08310054465 -> 838.015231637391
- link base_link: mass 2.2521398120105 -> 2.25213983841171
- link gripper_body: mass 0.833018335285825 -> 0.933264814357233
- link gripper_finger1: mass 0.0694658380950057 -> 0.0233180451311379
- link gripper_finger2: mass 0.0694658380901624 -> 0.023318045131138
- link gripper_tool1: mass 0.0524980209707732 -> 0.0524980209707729
- link gripper_tool2: mass 0.0524980209707734 -> 0.052498020970773
- link link1: mass 3.38715574374258 -> 3.38716123949166
- link link2: mass 10.3635830804756 -> 10.3635885023069
- link link3: mass 5.05083810344374 -> 5.05083741641896
- link link4: mass 0.809634503765035 -> 0.809634247265308
- link link5: mass 0.822358154530824 -> 0.822358399005338
- link link6: mass 0.23767801504912 -> 0.237678022472349
Joints:
- removed joint base_obstacle_fixed
- removed joint base_plate_pick_fixed
- removed joint base_plate_place_fixed
- removed joint slide_finger1
- removed joint slide_finger2
- added joint base_pick_fixed: type fixed, parent base_link, child pick, origin xyz=0 0 0 rpy=0 0 0, axis 0 0 0
- added joint base_plate_fixed: type fixed, parent base_link, child place, origin xyz=0 0 0 rpy=0 0 0, axis 0 0 0
- added joint base_table_fixed: type fixed, parent base_link, child table, origin xyz=0 0 0 rpy=0 0 0, axis 0 0 0
- added joint gripper_cam_fixed: type fixed, parent gripper_body, child cam, origin xyz=0 -0.13845 -0.0685 rpy=1.5708 0 0, axis 0 0 0
- added joint pick_circle_fixed: type fixed, parent pick, child pick_circle, origin xyz=0.23709 -0.71828 -0.068 rpy=0 0 0, axis 0 0 0
- added joint pick_cross_fixed: type fixed, parent pick, child pick_cross, origin xyz=0.16702 -0.80412 -0.068 rpy=0 0 0, axis 0 0 0
- added joint pick_rectangle_fixed: type fixed, parent pick, child pick_rectangle, origin xyz=0.16748 -0.60831 -0.068 rpy=0 0 0, axis 0 0 0
- added joint place_circle_rixed: type fixed, parent place, child place_circle, origin xyz=-0.16925 -0.84711 -0.078 rpy=0 0 0, axis 0 0 0
- added joint place_cross_fixed: type fixed, parent place, child place_cross, origin xyz=-0.28511 -0.67677 -0.078 rpy=0 0 0, axis 0 0 0
- added joint place_rectangle_fixed: type fixed, parent place, child place_rectangle, origin xyz=-0.15072 -0.71284 -0.078 rpy=0 0 0, axis 0 0 0
- added joint s1: type prismatic, parent gripper_body, child gripper_tool1, origin xyz=0 -0.0962 0 rpy=0 0 0, axis 1 0 0, limit lower=0 upper=0.04 effort=10 velocity=100
- added joint s2: type prismatic, parent gripper_body, child gripper_tool2, origin xyz=0 -0.0962 0 rpy=0 0 0, axis -1 0 0, limit lower=0 upper=0.04 effort=10 velocity=100
- joint base_fixed: limit lower=0 upper=0 effort=0 velocity=0 -> (none)
- joint link6_gripper_fixed: limit lower=-6.15 upper=6.15 effort=10 velocity=100 -> (none); origin xyz=0 0 -0.1148 rpy=1.5708 0.0070497 0 -> xyz=0 0 -0.1148 rpy=1.5708 0 0
- joint q1: limit lower=-6.15 upper=6.15 effort=10 velocity=100 -> lower=-6.3 upper=6.3 effort=10 velocity=100
- joint q2: limit lower=-6.15 upper=6.15 effort=10 velocity=100 -> lower=-6.3 upper=6.3 effort=10 velocity=100
- joint q3: limit lower=-6.15 upper=6.15 effort=10 velocity=100 -> lower=-6.3 upper=6.3 effort=10 velocity=100
- joint q4: limit lower=-6.15 upper=6.15 effort=10 velocity=100 -> lower=-6.3 upper=6.3 effort=10 velocity=100
- joint q5: limit lower=-6.15 upper=6.15 effort=10 velocity=100 -> lower=-6.3 upper=6.3 effort=10 velocity=100; origin xyz=0 0 -0.11715 rpy=1.5708 0.0070497 1.5708 -> xyz=0 0 -0.11715 rpy=1.5708 0 1.5708
- joint q6: limit lower=-6.15 upper=6.15 effort=10 velocity=100 -> lower=-6.3 upper=6.3 effort=10 velocity=100; origin xyz=0 0 0.11715 rpy=-1.5708 0 0.0070497 -> xyz=0 0 0.11715 rpy=-1.5708 0 0

Commit message: simulator 작업 중

File: keti_sdk_simulator/keti_robot_description/urdf/keti_robot_description.urdf (robot description, URDF)
Before this commit: robot keti_robot_arm, 23 links, 22 joints
Links:
- removed link gripper_body
- removed link gripper_finger1
- removed link gripper_finger2
- removed link gripper_tool1
- removed link gripper_tool2
- removed link pick
- removed link pick_circle
- removed link pick_cross
- removed link pick_rectangle
- removed link place
- removed link place_circle
- removed link place_cross
- removed link place_rectangle
- added link cage, mass 48.96; collision mesh filename=package://keti_robot_description/meshes/cage.STL; visual mesh filename=package://keti_robot_description/meshes/cage.STL
- added link cam_optical
- added link end
- added link gripper, mass 0.353450939027098; collision mesh filename=package://keti_robot_description/meshes/gripper.STL; visual mesh filename=package://keti_robot_description/meshes/gripper.STL
- added link gripper_cam_jig, mass 0.363809799934884; collision mesh filename=package://keti_robot_description/meshes/gripper_cam_jig.STL; visual mesh filename=package://keti_robot_description/meshes/gripper_cam_jig.STL
- added link tooltip1, mass 0.0737973344451048; collision mesh filename=package://keti_robot_description/meshes/tooltip1.STL; visual mesh filename=package://keti_robot_description/meshes/tooltip1.STL
- added link tooltip2, mass 0.0737973344451051; collision mesh filename=package://keti_robot_description/meshes/tooltip2.STL; visual mesh filename=package://keti_robot_description/meshes/tooltip2.STL
- added link world
- link base: mass 838.015231637391 -> 2.2652251953819
- link base_link: mass 2.25213983841171 -> 856.710523085829
- link cam: mass 0.0224324424296924 -> 0.0326887265041798
- link link1: mass 3.38716123949166 -> 3.38760416330855
- link link2: mass 10.3635885023069 -> 10.3582396210808
- link link3: mass 5.05083741641896 -> 5.05188870959058
- link link4: mass 0.809634247265308 -> 0.80963566860197
- link link5: mass 0.822358399005338 -> 0.822358205233283
- link link6: mass 0.237678022472349 -> 0.228532944621864
- link table: mass 361.6 -> 54.316
Joints:
- removed joint base_pick_fixed
- removed joint base_plate_fixed
- removed joint base_table_fixed
- removed joint gripper_cam_fixed
- removed joint link6_gripper_fixed
- removed joint pick_circle_fixed
- removed joint pick_cross_fixed
- removed joint pick_rectangle_fixed
- removed joint place_circle_rixed
- removed joint place_cross_fixed
- removed joint place_rectangle_fixed
- removed joint tool_finger1_fixed
- removed joint tool_finger2_fixed
- added joint base_table: type fixed, parent base_link, child table, origin xyz=-0.018106 -0.73131 0.017 rpy=0 0 -2.1411E-05, axis 0 0 0
- added joint cam_joint: type fixed, parent cam, child cam_optical, origin xyz=0 0 0.02495 rpy=-1.5708 -1.5708 0, axis 0 0 0
- added joint jig_cam: type fixed, parent gripper_cam_jig, child cam, origin xyz=-0.0583225279657438 0 -0.0820000000000001 rpy=3.14159265358979 0 1.5707963267949, axis 0 0 0
- added joint jig_gripper: type fixed, parent gripper_cam_jig, child gripper, origin xyz=0 0 -0.0658 rpy=0 0 0, axis 0 0 0
- added joint link6_end: type fixed, parent link6, child end, origin xyz=0 0 -0.1153 rpy=1.5708 -1.5708 0, axis 0 0 0
- added joint link6_jig: type fixed, parent link6, child gripper_cam_jig, origin xyz=0 0 -0.1183 rpy=0 0 2.4958, axis 0 0 0
- added joint table_cage: type fixed, parent table, child cage, origin xyz=0 0 0.803 rpy=0 0 0, axis 0 0 0
- added joint world_base: type fixed, parent world, child base_link, origin xyz=0 0 0 rpy=0 0 0, axis 0 0 0
- joint base_fixed: origin xyz=0 0 0 rpy=0 0 0 -> xyz=0 0 0.803 rpy=0 0 0
- joint q1: limit lower=-6.3 upper=6.3 effort=10 velocity=100 -> lower=-6.28 upper=6.28 effort=100 velocity=10; origin xyz=0 0 0 rpy=0 0 0 -> xyz=0 0 0 rpy=0 0 -1.5708; parent base_link -> base
- joint q2: limit lower=-6.3 upper=6.3 effort=10 velocity=100 -> lower=-6.28 upper=6.28 effort=100 velocity=10; origin xyz=0 0 0.198 rpy=-1.5708 0 0 -> xyz=0 0 0.197 rpy=1.5708 -1.5708 3.1416
- joint q3: limit lower=-6.3 upper=6.3 effort=10 velocity=100 -> lower=-6.28 upper=6.28 effort=100 velocity=10; origin xyz=0 -0.6127 -0.1875 rpy=0 0 -1.5708 -> xyz=0.6127 0 -0.1875 rpy=0 0 1.5708
- joint q4: limit lower=-6.3 upper=6.3 effort=10 velocity=100 -> lower=-6.28 upper=6.28 effort=100 velocity=10
- joint q5: limit lower=-6.3 upper=6.3 effort=10 velocity=100 -> lower=-6.28 upper=6.28 effort=100 velocity=10; origin xyz=0 0 -0.11715 rpy=1.5708 0 1.5708 -> xyz=0 0 -0.11715 rpy=0 -1.5708 -3.1416
- joint q6: limit lower=-6.3 upper=6.3 effort=10 velocity=100 -> lower=-6.28 upper=6.28 effort=100 velocity=10; origin xyz=0 0 0.11715 rpy=-1.5708 0 0 -> xyz=0 0 0.11715 rpy=1.5708 -1.5708 -3.1416
- joint s1: axis 1 0 0 -> 0 0 1; child gripper_tool1 -> tooltip1; limit lower=0 upper=0.04 effort=10 velocity=100 -> lower=0 upper=0.04 effort=100 velocity=10; origin xyz=0 -0.0962 0 rpy=0 0 0 -> xyz=0 0.041 -0.0608 rpy=1.5708 -1.5708 0; parent gripper_body -> gripper
- joint s2: axis -1 0 0 -> 0 0 1; child gripper_tool2 -> tooltip2; limit lower=0 upper=0.04 effort=10 velocity=100 -> lower=0 upper=0.04 effort=100 velocity=10; origin xyz=0 -0.0962 0 rpy=0 0 0 -> xyz=0 -0.041 -0.0608 rpy=-1.5708 -1.5708 0; parent gripper_body -> gripper

Commit message: simulator update

File: keti_sdk_simulator/keti_robot_description/urdf/keti_robot_description.urdf (robot description, URDF)
Before this commit: robot keti_robot_description, 18 links, 17 joints
Links:
- added link guide, mass 0.78172; collision mesh filename=package://keti_robot_description/meshes/guide.STL; visual mesh filename=package://keti_robot_description/meshes/guide.STL
- added link guide_plate, mass 2.83099; collision mesh filename=package://keti_robot_description/meshes/guide_plate.STL; visual mesh filename=package://keti_robot_description/meshes/guide_plate.STL
- added link sample, mass 0.21697; collision mesh filename=package://keti_robot_description/meshes/sample.STL; visual mesh filename=package://keti_robot_description/meshes/sample.STL
- added link sample_box, mass 3.96050; collision mesh filename=package://keti_robot_description/meshes/sample_box.STL; visual mesh filename=package://keti_robot_description/meshes/sample_box.STL
- link base: mass 2.2652251953819 -> 856.710523085829; geometry collision mesh filename=package://keti_robot_description/meshes/base_link.STL; visual mesh filename=package://keti_robot_description/meshes/base_link.STL
- link base_link: mass 856.710523085829 -> 2.2652251953819; geometry collision mesh filename=package://keti_robot_description/meshes/base.STL; visual mesh filename=package://keti_robot_description/meshes/base.STL
Joints:
- added joint box_sample: type fixed, parent sample_box, child sample, origin xyz=0.03961 0.04829 0.010 rpy=1.5708 0 0, axis 0 0 0
- added joint cage_box: type fixed, parent cage, child sample_box, origin xyz=0.21961 0.01 0 rpy=0 0 0, axis 0 0 0
- added joint cage_plate: type fixed, parent cage, child guide_plate, origin xyz=-0.18189 0.025 0 rpy=1.5708 0 0, axis 0 0 0
- added joint plate_guide: type fixed, parent guide_plate, child guide, origin xyz=0.01888 0.018 -0.02292 rpy=0 0 0, axis 0 0 0
- joint base_fixed: origin xyz=0 0 0.803 rpy=0 0 0 -> xyz=0 0 -0.803 rpy=0 0 0
- joint base_table: parent base_link -> base
- joint q1: parent base -> base_link
- joint world_base: origin xyz=0 0 0 rpy=0 0 0 -> xyz=0 0 0.803 rpy=0 0 0

Commit message: movel error fixed

File: keti_sdk_simulator/keti_robot_description/urdf/keti_robot_description.urdf (robot description, URDF)
Before this commit: robot keti_robot_description, 22 links, 21 joints
Joints:
- joint link6_end: origin xyz=0 0 -0.1153 rpy=1.5708 -1.5708 0 -> xyz=0 0 -0.1153 rpy=1.5708 0 1.5708

File: keti_sdk_simulator/keti_robot_moveit_config/config/gazebo_keti_robot_description.urdf (robot description, URDF)
Before this commit: robot keti_robot_description, 22 links, 21 joints
Joints:
- joint link6_end: origin xyz=0 0 -0.1153 rpy=1.5708 -1.5708 0 -> xyz=0 0 -0.1153 rpy=1.5708 0 1.5708
